File: _autosave-MAB19.kicad_pcb (KiCad board)
At the start: 2 copper layers, 84 parts, among them J1 Screw_Terminal_01x02, J2 Screw_Terminal_01x03, J401 USART, J601 RJ45, J602 RJ45, K1 coil: 12VDC, contact: 125V/10A, Q1 BCV27, U1 4N25, U201 MCP2551-I/SN, U202 MCP2515-xSO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

Commit message: Adicionado safe zone para separar os GNDs
Parts:
- C1, C2, C3, C4, D1, D2, D3, Q1, R1, R2, R3, R4, R5, R6, R7, TP1, TP2, TP3, TP4, TP5, U1: moved to B.Cu
- moved D3 147.8 mm to (68.4, 82.6)
- moved D1 141.9 mm to (60.8, 76.9)
- moved D2 141.8 mm to (56.2, 76.7)
- moved Q1 141.2 mm to (50.5, 76.1)
- moved R6 139.8 mm to (55.4, 74.6)
- moved C1 118.3 mm to (116.8, 95.2), turned to 270 degrees
- moved R3 117.0 mm to (89.5, 86.0)
- moved C2 107.0 mm to (80.6, 77.4)
- moved C4 107.0 mm to (76.9, 77.4)
- moved TP3 106.7 mm to (83.8, 77.1)
- moved C3 105.0 mm to (76.9, 75.4)
- moved TP5 104.7 mm to (80.0, 75.1)
- moved TP1 104.2 mm to (119.4, 92.7)
- moved TP4 102.8 mm to (76.3, 73.2)
- moved R2 99.8 mm to (71.7, 69.8)
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Routing:
- net GND: track 79.5 -> 106.8 mm
- net Net-(C1-Pad1): track 0.00 -> 21.7 mm
- net /MCU/ON_OFF_PUMP: track 0.00 -> 21.1 mm
- net +5V: track 187.6 -> 170.6 mm
- added copper zone on B.Cu, net GND
