File: MAB19.sch (KiCad schematic (older format))
At the start: 6 parts, among them J1 Screw_Terminal_01x02, J2 Screw_Terminal_01x03

Commit message: First version PCB
Connections:
- net GNDPWR: now also J1.2 (Pin_2); no longer J1.1 (Pin_1)
- net filter/Vin: now also J1.1 (Pin_1); no longer J1.2 (Pin_2)
Changed lines of the file:
@@
 EESchema Schematic File Version 4
+LIBS:MAB19-cache
 EELAYER 26 0
 EELAYER END
@@
 F3 "+5V_OUT" O L 7750 3250 60
 F4 "+18V_IN" I R 8800 3150 60
-F5 "+18V_OUT" I L 7750 3150 60
 $EndSheet
 $Sheet
@@
 L Connector:Screw_Terminal_01x02 J1
 U 1 1 5C901A4D
-P 1500 6650
-F 0 "J1" H 1420 6325 50  0000 C CNN
-F 1 "Screw_Terminal_01x02" H 1420 6416 50  0000 C CNN
-F 2 "TerminalBlock:TerminalBlock_bornier-2_P5.08mm" H 1500 6650 50  0001 C CNN
-F 3 "~" H 1500 6650 50  0001 C CNN
-	1    1500 6650
-	-1   0    0    1
-$EndComp
-Wire Wire Line
+P 1500 6550
+F 0 "J1" H 1420 6225 50  0000 C CNN
+F 1 "Screw_Terminal_01x02" H 1420 6316 50  0000 C CNN
+F 2 "TerminalBlock:TerminalBlock_bornier-2_P5.08mm" H 1500 6550 50  0001 C CNN
+F 3 "~" H 1500 6550 50  0001 C CNN
+	1    1500 6550
+	-1   0    0    -1
+$EndComp
+Wire Wire Line
