File: canbus.sch (KiCad schematic (older format))
At the start: 21 parts, among them U201 MCP2551-I/SN, U202 MCP2515-xSO, Y201 16MHz

Commit message: First version PCB
Parts:
- U202: symbol Interface_CAN_LIN:MCP2515-xSO -> MAB19-rescue:MCP2515-xSO-Interface_CAN_LIN
Changed lines of the file:
@@
 EESchema Schematic File Version 4
+LIBS:MAB19-cache
 EELAYER 26 0
 EELAYER END
@@
 Connection ~ 5550 4300
 $Comp
-L Interface_CAN_LIN:MCP2515-xSO U202
+L MAB19-rescue:MCP2515-xSO-Interface_CAN_LIN U202
 U 1 1 5BE69763
 P 4300 3700
+AR Path="/5BE69763" Ref="U202"  Part="1"
+AR Path="/5AABFC1B/5BE69763" Ref="U202"  Part="1"
 F 0 "U202" H 3850 4450 50  0000 C CNN
 F 1 "MCP2515-xSO" H 4650 2950 50  0000 C CNN
