File: pump_driver.sch (KiCad schematic (older format))
At the start: 24 parts, among them K1 coil: 12VDC, contact: 125V/10A, Q1 BCV27, U1 4N25

Commit message: First version PCB
Parts:
- added JP1: SolderJumper_3_Bridged12, Jumper:SolderJumper-3_P1.3mm_Bridged2Bar12_Pad1.0x1.5mm_NumberLabels, symbol Jumper:SolderJumper_3_Bridged12
Connections:
- net +Pump: now also JP1.2 (C); no longer K1.3
- net at K1.4: now also JP1.3 (B)
- new net: JP1.1 (A), K1.3
- no-connect marks 1 -> 0
Changed lines of the file:
@@
 EESchema Schematic File Version 4
+LIBS:MAB19-cache
 EELAYER 26 0
 EELAYER END
@@
 Wire Wire Line
 	5500 4750 5900 4750
-Wire Wire Line
-	7750 3800 7750 3850
 $Comp
 L Device:D_Small_ALT D4
@@
 	6650 4750 6650 4850
 Connection ~ 6650 4750
-NoConn ~ 7550 3800
 Wire Wire Line
 	6650 3100 6650 3150
@@
 	7750 4200 7750 4350
 Wire Wire Line
-	7750 3850 7750 4000
-Connection ~ 7750 3850
-Wire Wire Line
-	7750 3850 8150 3850
-Wire Wire Line
-	8150 4150 8150 3850
+	8150 4150 8150 4000
 Connection ~ 8150 3850
 Connection ~ 8150 4750
@@
 Wire Wire Line
 	7025 4750 7750 4750
+$Comp
+L Jumper:SolderJumper_3_Bridged12 JP1
+U 1 1 5C90C600
+P 7650 3850
+F 0 "JP1" H 7650 4055 50  0000 C CNN
+F 1 "SolderJumper_3_Bridged12" H 7650 3964 50  0000 C CNN
+F 2 "Jumper:SolderJumper-3_P1.3mm_Bridged2Bar12_Pad1.0x1.5mm_NumberLabels" H 7650 3850 50  0001 C CNN
+F 3 "~" H 7650 3850 50  0001 C CNN
+	1    7650 3850
+	-1   0    0    -1
+$EndComp
+Wire Wire Line
+	7750 3800 7850 3800
+Wire Wire Line
+	7850 3800 7850 3850
+Wire Wire Line
+	7550 3800 7450 3800
+Wire Wire Line
+	7450 3800 7450 3850
+Wire Wire Line
+	7650 4000 7750 4000
+Wire Wire Line
+	7750 4000 8150 4000
+Connection ~ 7750 4000
+Connection ~ 8150 4000
+Wire Wire Line
+	8150 4000 8150 3850
 $EndSCHEMATC
