File: supplies.sch (KiCad schematic (older format))
At the start: 7 parts, among them U501 LM7805

Commit message: First version PCB
Connections:
- net +18V_OUT: no longer names the net of C501.1, C502.1, F501.2, U501.1 (VI)
Changed lines of the file:
@@
 EESchema Schematic File Version 4
+LIBS:MAB19-cache
 EELAYER 26 0
 EELAYER END
 $Descr A4 11693 8268
 encoding utf-8
-Sheet 5 7
+Sheet 4 7
 Title ""
 Date ""
@@
 Wire Wire Line
 	4600 3950 4650 3950
-Text HLabel 6650 3550 2    60   Input ~ 0
-+18V_OUT
-Wire Wire Line
-	5200 3550 5200 3950
-Wire Wire Line
-	5200 3550 6650 3550
-Connection ~ 5200 3550
-Wire Wire Line
-	5200 3450 5200 3550
 $Comp
 L power:PWR_FLAG #FLG0501
@@
 	-1   0    0    1
 $EndComp
+Wire Wire Line
+	5200 3450 5200 3950
 $EndSCHEMATC
